File: pcb/curio.kicad_sch (KiCad schematic)
At the start: 29 parts, among them J1 TagConnect, J2 QUICK, SW1 SW_Push, U1 STM32G0xxFx, U2 TSSP58038, U3 LCD12864

Commit message: rev 0x02
Connections:
- net LCD_BLK: now also U1.13 (PA6); no longer U1.14 (PA7)
- net LCD_SDA: now also U1.14 (PA7); no longer U1.13 (PA6)
Changed lines of the file:
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@@
   (title_block
     (title "Curio")
-    (rev "0x01")
+    (rev "0x02")
   )
   (junction (at 194.31 60.96) (diameter 0) (color 0 0 0 0)
@@
     (effects (font (size 1.27 1.27)) (justify right bottom))
   )
-  (label "LCD_SDA" (at 105.41 76.2 0) (fields_autoplaced)
+  (label "LCD_SDA" (at 105.41 78.74 0) (fields_autoplaced)
     (effects (font (size 1.27 1.27)) (justify left bottom))
   )
@@
     (effects (font (size 1.27 1.27)) (justify left bottom))
   )
-  (label "LCD_BLK" (at 105.41 78.74 0) (fields_autoplaced)
-    (effects (font (size 1.27 1.27)) (justify left bottom))
-  )
+  (label "LCD_BLK" (at 105.41 76.2 0) (fields_autoplaced)
+    (effects (font (size 1.27 1.27)) (justify left bottom))
+  )
