File: pcb/curio.kicad_sch (KiCad schematic)
At the start: 29 parts, among them J1 TagConnect, J2 QUICK, SW1 SW_Push, U1 STM32G0xxFx, U2 TSSP58038, U3 LCD12864

Commit message: update hal version
Parts:
- BT1: value Battery_Cell -> CR2030; footprint (none) -> curio:BatteryHolder-Lynx-BAT-HLD-001
- C1: value C -> 10uF
- C2, C3, C4, C5: renamed from C1; value C -> 100nF
- C6: renamed from C1; value C -> 10uF
- J2: value QUICK -> Qwiic
- R1: value R -> 10K
- R10, R9: renamed from R1; value R -> 10K
- R2: renamed from R1; value R -> 0R
- R3, R4, R8: renamed from R1; value R -> 190R
- R5, R6: renamed from R1; value R -> 4K7
- R7: renamed from R1; value R -> 1K
- RV1: value R_Potentiometer_Dual_Separate -> Thumbstick; footprint (none) -> curio:Thumbstick
- SW1: value SW_Push -> Reset; footprint Resistor_SMD:R_1206_3216Metric -> Resistor_SMD:R_1206_3216Metric_Pad1.30x1.75mm_HandSolder
- SW2: renamed from SW1; value SW_Push -> BTN_A; footprint Resistor_SMD:R_1206_3216Metric -> Button_Switch_SMD:SW_DIP_SPSTx01_Slide_6.7x4.1mm_W6.73mm_P2.54mm_LowProfile_JPin
- SW3: renamed from SW1; value SW_Push -> BTN_B; footprint Resistor_SMD:R_1206_3216Metric -> Button_Switch_SMD:SW_DIP_SPSTx01_Slide_6.7x4.1mm_W6.73mm_P2.54mm_LowProfile_JPin
- renumbered FB1 to FB2
