File: pcb/curio.kicad_pcb (KiCad board)
At the start: 4 copper layers, 76.2 x 25.4 mm, 31 parts, among them J1 TagConnect, J2 Qwiic, SW1 Reset, SW2 BTN_A, SW3 BTN_B, U1 STM32G0xxFx, U2 TSSP58038, U3 LCD12864

Commit message: rev 0x02
Parts:
- moved R2 0.51 mm to (125.1, 98.9)
Connections:
- U1 pad 13: /LCD_SDA -> /LCD_BLK
- U1 pad 14: /LCD_BLK -> /LCD_SDA
Routing:
- net /LCD_SDA: track 26.8 -> 28.4 mm
- net /LCD_A0: track 29.6 -> 30.4 mm
